Commit message: Update_2 5_11

File: robot_description/imu.xacro (robot description, xacro)
@@ -12,16 +12,64 @@
                 <box size="0.1 0.1 0.02" />
             </geometry>
-            <material name="dark"/>
+            <material name="grey"/>
         </visual>
         <collision>
             <origin xyz="0.0 0.0 0.0" rpy="0.0 0.0 0.0"/>
             <geometry>
-                <box size="0.2 0.2 0.2" />
+                <box size="0.2 0.2 0.02" />
             </geometry>
         </collision>
     </link>
-    <!-- <gazebo>
-        <plugin name="marinero_imu_link" filename="">
-        </plugin>
-    </gazebo> -->
+    <gazebo reference="imu_link">
+        <gravity>true</gravity>
+        <sensor name="imu_sensor" type="imu">
+            <always_on>true</always_on>
+            <update_rate>100</update_rate>
+            <visualize>true</visualize>
+            <plugin filename="libgazebo_ros_imu_sensor.so" name="imu_plugin">
+                <ros>
+                    <remapping>~/out:=/marinero/imu_sensor</remapping>
+                </ros>
+                <body_name>imu_link</body_name>
+                <update_rate_hz>10.0</update_rate_hz>
+                <gaussian_noise>0.0</gaussian_noise>
+                <xyz_offset>0 0 0</xyz_offset>
+                <rpy_offset>0 0 0</rpy_offset>
+                <frame_name>imu_link</frame_name>
+                <initial_orientation_as_reference>false</initial_orientation_as_reference>
+            </plugin>
+            <pose>0 0 0 0 0 0</pose>
+        </sensor>
+    </gazebo>
+    <joint name="gps_joint" type="fixed">
+        <parent link="base_link"/>
+        <child link="gps_link"/>
+        <origin xyz="0 0 0.32" rpy="0 0 0"/>
+    </joint>
+    <link name="gps_link">
+        <visual>
+            <origin xyz="0.0 0.0 0.0" rpy="0.0 0.0 0.0"/>
+            <geometry>
+                <box size="0.1 0.1 0.02" />
+            </geometry>
+            <material name="white"/>
+        </visual>
+        <collision>
+            <origin xyz="0.0 0.0 0.0" rpy="0.0 0.0 0.0"/>
+            <geometry>
+                <box size="0.2 0.2 0.02" />
+            </geometry>
+        </collision>
+    </link>
+    <gazebo reference="gps_link">
+        <sensor name="gps_sensor" type="gps">
+            <always_on>true</always_on>
+            <update_rate>30</update_rate>
+            <plugin name="my_gps_plugin" filename="libgazebo_ros_gps_sensor.so">
+                <ros>
+                    <remapping>~/out:=/marinero/gps_sensor</remapping>
+                </ros>
+            </plugin>
+        </sensor>
+    </gazebo>
 </robot>

File: robot_description/lidar.xacro (robot description, xacro)
@@ -46,25 +46,25 @@
         <sensor name="3D_lidar" type="ray">
             <pose>0 0 0 0 0 0</pose>
-            <update_rate>10.0</update_rate>
+            <update_rate>7.5</update_rate>
             <visualize>false</visualize>
             <ray>
                 <scan>
                     <horizontal>
+                        <samples>180.0</samples>
+                        <resolution>1.0</resolution>
+                        <min_angle>${-pi/2}</min_angle>
+                        <max_angle>${pi/2}</max_angle>
+                    </horizontal>
+                    <vertical>
                         <samples>100.0</samples>
                         <resolution>1.0</resolution>
-                        <min_angle>${-2*pi/3}</min_angle>
-                        <max_angle>${2*pi/3}</max_angle>
-                    </horizontal>
-                    <vertical>
-                        <samples>85.0</samples>
-                        <resolution>1.0</resolution>
-                        <min_angle>-0.1</min_angle>
-                        <max_angle>0.8</max_angle>
+                        <min_angle>-0.25</min_angle>
+                        <max_angle>1.25</max_angle>
                     </vertical>
                 </scan>
                 <range>
                     <min>0.5</min>
-                    <max>10.0</max>
-                    <resolution>0.001</resolution>
+                    <max>5.0</max>
+                    <resolution>0.005</resolution>
                 </range>
             </ray>

File: robot_description/marinero_robot.urdf.xacro (robot description, xacro)
@@ -1,21 +1,22 @@
 <?xml version="1.0" ?>
 <robot xmlns:xacro="http://www.ros.org/wiki/xacro" name="marinero">
-  <xacro:arg name="sim_mode" default="true"/>
-  <xacro:arg name="use_ros2_control" default="true"/>
-  <xacro:arg name="use_4wis4wid" default="true"/>
-  <xacro:include filename="materials.xacro" />
-  <xacro:include filename="lidar.xacro" />
-  <xacro:include filename="marinero_camera.xacro" />
-  <xacro:if value="$(arg use_4wis4wid)">
-      <xacro:include filename="robot_core_4WIS4WID.xacro" />
-  </xacro:if>
-  <xacro:unless value="$(arg use_4wis4wid)">
-      <xacro:include filename="robot_core.xacro" />
-  </xacro:unless>
-  <xacro:if value="$(arg use_ros2_control)">
-      <xacro:include filename="ros2_control.xacro" />
-  </xacro:if>
-  <xacro:unless value="$(arg use_ros2_control)">
-      <xacro:include filename="gazebo_control.xacro" />
-  </xacro:unless>
+    <xacro:arg name="sim_mode" default="true"/>
+    <xacro:arg name="use_ros2_control" default="true"/>
+    <xacro:arg name="use_4wis4wid" default="true"/>
+    <xacro:include filename="materials.xacro" />
+    <xacro:include filename="imu.xacro" />
+    <xacro:include filename="lidar.xacro" />
+    <xacro:include filename="marinero_camera.xacro" />
+    <xacro:if value="$(arg use_4wis4wid)">
+        <xacro:include filename="robot_core_4WIS4WID.xacro" />
+    </xacro:if>
+    <xacro:unless value="$(arg use_4wis4wid)">
+        <xacro:include filename="robot_core.xacro" />
+    </xacro:unless>
+    <xacro:if value="$(arg use_ros2_control)">
+        <xacro:include filename="ros2_control.xacro" />
+    </xacro:if>
+    <xacro:unless value="$(arg use_ros2_control)">
+        <xacro:include filename="gazebo_control.xacro" />
+    </xacro:unless>
 </robot>

File: robot_description/rsp_marinero_robot.urdf.xacro (robot description, xacro)
@@ -2,4 +2,5 @@
 <robot xmlns:xacro="http://www.ros.org/wiki/xacro" name="marinero">
   <xacro:include filename="materials.xacro" />
+  <xacro:include filename="imu.xacro" />
   <xacro:include filename="lidar.xacro" />
   <xacro:include filename="marinero_camera.xacro" />
