Commit message: Update 11_12

File: robot_description/gazebo_control.xacro (robot description, xacro)
@@ -107,6 +107,6 @@
             <robot_base_frame>base_link</robot_base_frame>
             <ros>
-                <!-- <argument>/cmd_vel:=/skid_steer/cmd_vel_joy</argument> -->
-                <argument>/odom:=/marinero/odom</argument>
+                <namespace>/</namespace>
+                <remapping>odom:=/marinero/odom</remapping>
             </ros>
             <covariance_x>0.001</covariance_x>

File: robot_description/lidar.xacro (robot description, xacro)
@@ -24,13 +24,7 @@
         </visual>
         <collision>
-            <origin xyz="0 0 -0.025" />
-            <geometry>
-                <cylinder radius="${lidar_radius}" length="${lidar_length}"/>
-            </geometry>
-        </collision>
-        <collision>
             <origin xyz="0 0 0" />
             <geometry>
-                <sphere radius="${lidar_radius - 0.01}"/>
+                <cylinder radius="${lidar_radius*1.15}" length="${lidar_length*2}"/>
             </geometry>
         </collision>
@@ -79,5 +73,5 @@
     </gazebo>
     <!-- 2D LIDAR -->
-    <!-- <gazebo reference="lidar_link">
+    <gazebo reference="lidar_link">
         <sensor name="2D_lidar" type="gpu_ray">
             <pose> 0 0 0 0 0 0 </pose>
@@ -95,5 +89,5 @@
                 <range>
                     <min>0.75</min>
-                    <max>10</max>
+                    <max>15</max>
                     <resolution>0.01</resolution>
                 </range>
@@ -107,4 +101,4 @@
             </plugin>
         </sensor>
-    </gazebo> -->
+    </gazebo>
 </robot>

File: robot_description/marinero_camera.xacro (robot description, xacro)
@@ -13,5 +13,5 @@
         <!-- <dynamics damping="0.1" /> -->
         <dynamics damping="0.2" friction="5.0" />
-    </joint>i
+    </joint>
     <link name="camera_base">
         <visual>
@@ -21,9 +21,9 @@
             </geometry>
             <material name="dark"/>
-        </visual>k
+        </visual>
         <collision>
-            <origin xyz="0.0 0.0 0.0"/>
+            <origin xyz="0.0 0.0 0.095"/>
             <geometry>
-                <mesh filename="file:///home/albert/marinero_ws/src/marinero_simulations/robot_description/meshes/Camera_Base.stl" scale="1.0 1.0 1.0"/>
+                <cylinder length="0.192" radius="0.1"/>
             </geometry>
         </collision>
@@ -59,7 +59,7 @@
         </visual>
         <collision>
-            <origin xyz="0.0 0.0 0.0"/>
+            <origin xyz="-0.09 0.0 0.0"/>
             <geometry>
-                <mesh filename="file:///home/albert/marinero_ws/src/marinero_simulations/robot_description/meshes/Camera_L.stl" scale="1.0 1.0 1.0"/>
+                <cylinder length="0.16" radius="0.066"/>
             </geometry>
         </collision>
@@ -107,7 +107,7 @@
         </visual>
         <collision>
-            <origin xyz="0.0 0.0 0.0"/>
+            <origin xyz="0.09 0.0 0.0"/>
             <geometry>
-                <mesh filename="file:///home/albert/marinero_ws/src/marinero_simulations/robot_description/meshes/Camera_R.stl" scale="1.0 1.0 1.0"/>
+                <cylinder length="0.16" radius="0.066"/>
             </geometry>
         </collision>

File: robot_description/robot_core.xacro (robot description, xacro)
@@ -17,11 +17,23 @@
             <origin xyz="0.0 0.0 0.014" />
             <geometry>
-                <mesh filename="file:///home/albert/marinero_ws/src/marinero_simulations/robot_description/meshes/MARINERO_chassis.dae" scale="1.0 1.0 1.0" />
-            </geometry>
-        </visual>
-        <collision>
-            <origin xyz="0.0 0.0 0.1" />
-            <geometry>
-                <box size="0.6655 1.075 0.2"/>
+                <mesh filename="file:///home/albert/marinero_ws/src/marinero_simulations/robot_description/meshes/MARINERO_chassis_no_driving_assembly.dae" scale="1.0 1.0 1.0" />
+            </geometry>
+        </visual>
+        <collision>
+            <origin xyz="0.0 0.0 0.08" />
+            <geometry>
+                <box size="0.6656 1.077 0.165"/>
+            </geometry>
+        </collision>
+        <collision>
+            <origin xyz="0.0 -0.23 0.305"/>
+            <geometry>
+                    <cylinder length="0.29" radius="0.18"/>
+            </geometry>
+        </collision>
+        <collision>
+            <origin xyz="0.0 0.28 0.195" rpy="0 0 0"/>
+            <geometry>
+                    <box size="0.36 0.45 0.075"/>
             </geometry>
         </collision>

File: robot_description/robot_core_4WIS4WID.xacro (robot description, xacro)
@@ -17,11 +17,23 @@
             <origin xyz="0.0 0.0 0.014" />
             <geometry>
-                <mesh filename="file:///home/albert/marinero_ws/src/marinero_simulations/robot_description/meshes/MARINERO_chassis.dae" scale="1.0 1.0 1.0" />
-            </geometry>
-        </visual>
-        <collision>
-            <origin xyz="0.0 0.0 0.1" />
-            <geometry>
-                <box size="0.6655 1.075 0.2"/>
+                <mesh filename="file:///home/albert/marinero_ws/src/marinero_simulations/robot_description/meshes//MARINERO_chassis_no_driving_assembly.dae" scale="1.0 1.0 1.0" />
+            </geometry>
+        </visual>
+        <collision>
+            <origin xyz="0.0 0.0 0.08" />
+            <geometry>
+                <box size="0.6656 1.077 0.165"/>
+            </geometry>
+        </collision>
+        <collision>
+            <origin xyz="0.0 -0.23 0.305"/>
+            <geometry>
+                    <cylinder length="0.29" radius="0.18"/>
+            </geometry>
+        </collision>
+        <collision>
+            <origin xyz="0.0 0.28 0.195" rpy="0 0 0"/>
+            <geometry>
+                    <box size="0.36 0.45 0.075"/>
             </geometry>
         </collision>
@@ -92,4 +104,7 @@
         <dynamics friction="2.0"/>
     </joint>
+            <geometry>
+                <mesh filename="file:///home/albert/marinero_ws/src/marinero_simulations/robot_description/meshes/Camera_R.stl" scale="1.0 1.0 1.0"/>
+            </geometry>
     <link name="fl_wheel">
         <visual>

Commit message: Update 12_12

File: robot_description/gazebo_control.xacro (robot description, xacro)
@@ -84,5 +84,5 @@
         <plugin name="skid_steer_drive" filename="libgazebo_ros_diff_drive.so">
             <!-- Update rate -->
-            <update_rate>150</update_rate>
+            <update_rate>100</update_rate>
             <!-- Number of wheel pairs -->
             <num_wheel_pairs>2</num_wheel_pairs>
@@ -98,5 +98,5 @@
             <wheel_diameter>0.2032</wheel_diameter>
             <!-- limits -->
-            <max_wheel_torque>150.0</max_wheel_torque>
+            <max_wheel_torque>100.0</max_wheel_torque>
             <max_wheel_acceleration>7.0</max_wheel_acceleration>
             <!-- output -->
@@ -107,6 +107,5 @@
             <robot_base_frame>base_link</robot_base_frame>
             <ros>
-                <namespace>/</namespace>
-                <remapping>odom:=/marinero/odom</remapping>
+                <remapping>/odom:=/marinero/odom</remapping>
             </ros>
             <covariance_x>0.001</covariance_x>
@@ -118,5 +117,5 @@
         <plugin name="gazebo_ros_joint_state_publisher"
             filename="libgazebo_ros_joint_state_publisher.so">
-            <update_rate>150</update_rate>
+            <update_rate>200</update_rate>
             <joint_name>camera_base_joint</joint_name>
             <joint_name>left_camera_joint</joint_name>
@@ -127,5 +126,5 @@
         <plugin name="gazebo_ros_joint_pose_trajectory"
             filename="libgazebo_ros_joint_pose_trajectory.so">
-            <update_rate>150</update_rate>
+            <update_rate>200</update_rate>
         </plugin>
     </gazebo>

File: robot_description/lidar.xacro (robot description, xacro)
@@ -40,5 +40,5 @@
         <sensor name="3D_lidar" type="gpu_ray">
             <pose>0 0 0 0 0 0</pose>
-            <update_rate>15</update_rate>
+            <update_rate>15.0</update_rate>
             <visualize>false</visualize>
             <ray>
@@ -76,5 +76,5 @@
         <sensor name="2D_lidar" type="gpu_ray">
             <pose> 0 0 0 0 0 0 </pose>
-            <update_rate>15</update_rate>
+            <update_rate>20.0</update_rate>
             <visualize>false</visualize>
             <ray>

File: robot_description/marinero_camera.xacro (robot description, xacro)
@@ -12,5 +12,5 @@
             velocity="100" />
         <!-- <dynamics damping="0.1" /> -->
-        <dynamics damping="0.2" friction="5.0" />
+        <dynamics damping="10.0" friction="5.0" />
     </joint>
     <link name="camera_base">
@@ -48,5 +48,5 @@
             velocity="100" />
         <!-- <dynamics damping="1.0" friction="10.0" /> -->
-        <dynamics damping="0.2" friction="5.0" />
+        <dynamics damping="10.0" friction="5.0" />
     </joint>
     <link name="right_camera_link">
@@ -95,6 +95,5 @@
             effort="100"
             velocity="100" />
-        <!-- <dynamics damping="1.0" friction="10.0" /> -->
-        <dynamics damping="0.2" friction="5.0" />
+        <dynamics damping="10.0" friction="5.0" />
     </joint>
     <link name="left_camera_link">

Commit message: Update 17_12

File: robot_description/gazebo_control.xacro (robot description, xacro)
@@ -84,5 +84,5 @@
         <plugin name="skid_steer_drive" filename="libgazebo_ros_diff_drive.so">
             <!-- Update rate -->
-            <update_rate>100</update_rate>
+            <update_rate>150</update_rate>
             <!-- Number of wheel pairs -->
             <num_wheel_pairs>2</num_wheel_pairs>

File: robot_description/marinero_camera.xacro (robot description, xacro)
@@ -47,6 +47,5 @@
             effort="100"
             velocity="100" />
-        <!-- <dynamics damping="1.0" friction="10.0" /> -->
-        <dynamics damping="10.0" friction="5.0" />
+        <dynamics damping="10.0" friction="10.0" />
     </joint>
     <link name="right_camera_link">

Commit message: Update 20_12

File: robot_description/gazebo_control.xacro (robot description, xacro)
@@ -84,5 +84,5 @@
         <plugin name="skid_steer_drive" filename="libgazebo_ros_diff_drive.so">
             <!-- Update rate -->
-            <update_rate>150</update_rate>
+            <update_rate>200</update_rate>
             <!-- Number of wheel pairs -->
             <num_wheel_pairs>2</num_wheel_pairs>
@@ -117,5 +117,5 @@
         <plugin name="gazebo_ros_joint_state_publisher"
             filename="libgazebo_ros_joint_state_publisher.so">
-            <update_rate>200</update_rate>
+            <update_rate>100</update_rate>
             <joint_name>camera_base_joint</joint_name>
             <joint_name>left_camera_joint</joint_name>
@@ -126,5 +126,5 @@
         <plugin name="gazebo_ros_joint_pose_trajectory"
             filename="libgazebo_ros_joint_pose_trajectory.so">
-            <update_rate>200</update_rate>
+            <update_rate>100</update_rate>
         </plugin>
     </gazebo>

File: robot_description/imu.xacro (robot description, xacro)
@@ -65,5 +65,5 @@
         <sensor name="gps_sensor" type="gps">
             <always_on>true</always_on>
-            <update_rate>30</update_rate>
+            <update_rate>10</update_rate>
             <plugin name="my_gps_plugin" filename="libgazebo_ros_gps_sensor.so">
                 <ros>

File: robot_description/lidar.xacro (robot description, xacro)
@@ -36,6 +36,18 @@
         </xacro:inertial_sphere>
     </link>
+    <joint name="lidar_2D_joint" type="fixed">
+        <origin xyz="0.0 0.0 0.0" rpy="0.0 0.0 0.0"/>
+        <parent link="lidar_link"/>
+        <child link="lidar_2D_link"/>
+    </joint>
+    <link name="lidar_2D_link"></link>
+    <joint name="lidar_3D_joint" type="fixed">
+        <origin xyz="0.0 0.0 0.0" rpy="0.0 0.0 0.0"/>
+        <parent link="lidar_link"/>
+        <child link="lidar_3D_link"/>
+    </joint>
+    <link name="lidar_3D_link"></link>
     <!-- 3D LIDAR -->
-    <gazebo reference="lidar_link">
+    <gazebo reference="lidar_3D_link">
         <sensor name="3D_lidar" type="gpu_ray">
             <pose>0 0 0 0 0 0</pose>
@@ -67,14 +79,15 @@
                     <remapping>~/out:=/lidar_3D/scan</remapping>
                 </ros>
+                <update_rate>15.0</update_rate>
                 <output_type>sensor_msgs/PointCloud2</output_type>
-                <frame_name>lidar_link</frame_name>
+                <frame_name>lidar_3D_link</frame_name>
             </plugin>
         </sensor>
     </gazebo>
     <!-- 2D LIDAR -->
-    <gazebo reference="lidar_link">
+    <gazebo reference="lidar_2D_link">
         <sensor name="2D_lidar" type="gpu_ray">
             <pose> 0 0 0 0 0 0 </pose>
-            <update_rate>20.0</update_rate>
+            <update_rate>15.0</update_rate>
             <visualize>false</visualize>
             <ray>
@@ -97,6 +110,7 @@
                     <remapping>~/out:=/scan</remapping>
                 </ros>
+                <update_rate>15.0</update_rate>
                 <output_type>sensor_msgs/LaserScan</output_type>
-                <frame_name>lidar_link</frame_name>
+                <frame_name>lidar_2D_link</frame_name>
             </plugin>
         </sensor>

File: robot_description/ros2_control.xacro (robot description, xacro)
@@ -157,5 +157,5 @@
                 <remapping>odom:=/marinero/odom</remapping>
             </ros>
-            <frame_name>world</frame_name>
+            <frame_name>map</frame_name>
             <body_name>base_link</body_name>
             <update_rate>150</update_rate>
