Commit message: Update_21_02

File: robot_description/gazebo_control.xacro (robot description, xacro)
@@ -84,5 +84,5 @@
         <plugin name="skid_steer_drive" filename="libgazebo_ros_diff_drive.so">
             <!-- Update rate -->
-            <update_rate>200</update_rate>
+            <update_rate>100</update_rate>
             <!-- Number of wheel pairs -->
             <num_wheel_pairs>2</num_wheel_pairs>

File: robot_description/marinero_camera.xacro (robot description, xacro)
@@ -18,5 +18,5 @@
             <origin xyz="0.0 0.0 0.0" rpy="0 0 0"/>
             <geometry>
-                <mesh filename="file:///home/albert/marinero_ws/src/marinero_simulations/robot_description/meshes/Camera_Base.stl" scale="1.0 1.0 1.0"/>
+                <mesh filename="package://marinero_simulations/robot_description/meshes/Camera_Base.stl" scale="1.0 1.0 1.0"/>
             </geometry>
             <material name="dark"/>
@@ -53,5 +53,5 @@
             <origin xyz="0.0 0.0 0.0" rpy="0.0 0.0 0.0"/>
             <geometry>
-                <mesh filename="file:///home/albert/marinero_ws/src/marinero_simulations/robot_description/meshes/Camera_L.stl" scale="1.0 1.0 1.0"/>
+                <mesh filename="package://marinero_simulations/robot_description/meshes/Camera_L.stl" scale="1.0 1.0 1.0"/>
             </geometry>
             <material name="grey" />
@@ -100,5 +100,5 @@
             <origin xyz="0 0 0" rpy="0.0 0.0 0.0"/>
             <geometry>
-                <mesh filename="file:///home/albert/marinero_ws/src/marinero_simulations/robot_description/meshes/Camera_R.stl" scale="1.0 1.0 1.0"/>
+                <mesh filename="package://marinero_simulations/robot_description/meshes/Camera_R.stl" scale="1.0 1.0 1.0"/>
             </geometry>
             <material name="grey" />

File: robot_description/robot_core.xacro (robot description, xacro)
@@ -17,5 +17,5 @@
             <origin xyz="0.0 0.0 0.014" />
             <geometry>
-                <mesh filename="file:///home/albert/marinero_ws/src/marinero_simulations/robot_description/meshes/MARINERO_chassis_no_driving_assembly.dae" scale="1.0 1.0 1.0" />
+                <mesh filename="package://marinero_simulations/robot_description/meshes/MARINERO_chassis_no_driving_assembly.dae" scale="1.0 1.0 1.0" />
             </geometry>
         </visual>
@@ -60,5 +60,5 @@
             <origin xyz="0 0 0.1466" rpy="0 0 ${pi/2}"/>    <!-- xyz="0 0 ${0.156697-0.01}" -->
             <geometry>
-                <mesh filename="file:///home/albert/marinero_ws/src/marinero_simulations/robot_description/meshes/Wheel_Assembly.stl" scale="1.0 1.0 1.0" />
+                <mesh filename="package://marinero_simulations/robot_description/meshes/Wheel_Assembly.stl" scale="1.0 1.0 1.0" />
             </geometry>
             <material name="dark" />
@@ -102,5 +102,5 @@
             <origin xyz="0 0 0" rpy="0 0 0"/>
             <geometry>
-                <mesh filename="file:///home/albert/marinero_ws/src/marinero_simulations/robot_description/meshes/Wheel.stl" scale="1.0 1.0 1.0" />
+                <mesh filename="package://marinero_simulations/robot_description/meshes/Wheel.stl" scale="1.0 1.0 1.0" />
             </geometry>
             <material name="black"/>
@@ -129,5 +129,5 @@
             <origin xyz="0 0 0.1466" rpy="0 0 ${pi/2}"/>
             <geometry>
-                <mesh filename="file:///home/albert/marinero_ws/src/marinero_simulations/robot_description/meshes/Wheel_Assembly.stl" scale="1.0 1.0 1.0" />
+                <mesh filename="package://marinero_simulations/robot_description/meshes/Wheel_Assembly.stl" scale="1.0 1.0 1.0" />
             </geometry>
             <material name="dark" />
@@ -170,5 +170,5 @@
         <visual>
             <geometry>
-                <mesh filename="file:///home/albert/marinero_ws/src/marinero_simulations/robot_description/meshes/Wheel.stl" scale="1.0 1.0 1.0" />
+                <mesh filename="package://marinero_simulations/robot_description/meshes/Wheel.stl" scale="1.0 1.0 1.0" />
             </geometry>
             <material name="black"/>
@@ -197,5 +197,5 @@
             <origin xyz="0 0 0.1466" rpy="0 0 ${pi/2}"/>
             <geometry>
-                <mesh filename="file:///home/albert/marinero_ws/src/marinero_simulations/robot_description/meshes/Wheel_Assembly.stl" scale="1.0 1.0 1.0" />
+                <mesh filename="package://marinero_simulations/robot_description/meshes/Wheel_Assembly.stl" scale="1.0 1.0 1.0" />
             </geometry>
             <material name="dark" />
@@ -238,5 +238,5 @@
         <visual>
             <geometry>
-                <mesh filename="file:///home/albert/marinero_ws/src/marinero_simulations/robot_description/meshes/Wheel.stl" scale="1.0 1.0 1.0" />
+                <mesh filename="package://marinero_simulations/robot_description/meshes/Wheel.stl" scale="1.0 1.0 1.0" />
             </geometry>
             <material name="black"/>
@@ -265,5 +265,5 @@
             <origin xyz="0 0 0.1466" rpy="0 0 ${pi/2}"/>
             <geometry>
-                <mesh filename="file:///home/albert/marinero_ws/src/marinero_simulations/robot_description/meshes/Wheel_Assembly.stl" scale="1.0 1.0 1.0" />
+                <mesh filename="package://marinero_simulations/robot_description/meshes/Wheel_Assembly.stl" scale="1.0 1.0 1.0" />
             </geometry>
             <material name="dark" />
@@ -306,5 +306,5 @@
         <visual>
             <geometry>
-                <mesh filename="file:///home/albert/marinero_ws/src/marinero_simulations/robot_description/meshes/Wheel.stl" scale="1.0 1.0 1.0" />
+                <mesh filename="package://marinero_simulations/robot_description/meshes/Wheel.stl" scale="1.0 1.0 1.0" />
             </geometry>
             <material name="black"/>

File: robot_description/robot_core_4WIS4WID.xacro (robot description, xacro)
@@ -17,5 +17,5 @@
             <origin xyz="0.0 0.0 0.014" />
             <geometry>
-                <mesh filename="file:///home/albert/marinero_ws/src/marinero_simulations/robot_description/meshes//MARINERO_chassis_no_driving_assembly.dae" scale="1.0 1.0 1.0" />
+                <mesh filename="package://marinero_simulations/robot_description/meshes/MARINERO_chassis_no_driving_assembly.dae" scale="1.0 1.0 1.0" />
             </geometry>
         </visual>
@@ -66,5 +66,5 @@
             <origin xyz="0 0 0.1466" rpy="0 0 ${pi/2}"/>    <!-- xyz="0 0 ${0.156697-0.01}" -->
             <geometry>
-                <mesh filename="file:///home/albert/marinero_ws/src/marinero_simulations/robot_description/meshes/Wheel_Assembly.stl" scale="1.0 1.0 1.0" />
+                <mesh filename="package://marinero_simulations/robot_description/meshes/Wheel_Assembly.stl" scale="1.0 1.0 1.0" />
             </geometry>
             <material name="dark" />
@@ -105,5 +105,5 @@
     </joint>
             <geometry>
-                <mesh filename="file:///home/albert/marinero_ws/src/marinero_simulations/robot_description/meshes/Camera_R.stl" scale="1.0 1.0 1.0"/>
+                <mesh filename="package://marinero_simulations/robot_description/meshes/Camera_R.stl" scale="1.0 1.0 1.0"/>
             </geometry>
     <link name="fl_wheel">
@@ -111,5 +111,5 @@
             <origin xyz="0 0 0" rpy="0 0 0"/>
             <geometry>
-                <mesh filename="file:///home/albert/marinero_ws/src/marinero_simulations/robot_description/meshes/Wheel.stl" scale="1.0 1.0 1.0" />
+                <mesh filename="package://marinero_simulations/robot_description/meshes/Wheel.stl" scale="1.0 1.0 1.0" />
             </geometry>
             <material name="black"/>
@@ -147,5 +147,5 @@
             <origin xyz="0 0 0.1466" rpy="0 0 ${pi/2}"/>
             <geometry>
-                <mesh filename="file:///home/albert/marinero_ws/src/marinero_simulations/robot_description/meshes/Wheel_Assembly.stl"  scale="1.0 1.0 1.0" />
+                <mesh filename="package://marinero_simulations/robot_description/meshes/Wheel_Assembly.stl"  scale="1.0 1.0 1.0" />
             </geometry>
             <material name="dark" />
@@ -189,5 +189,5 @@
             <origin xyz="0 0 0" rpy="0 0 0"/>
             <geometry>
-                <mesh filename="file:///home/albert/marinero_ws/src/marinero_simulations/robot_description/meshes/Wheel.stl" scale="1.0 1.0 1.0" />
+                <mesh filename="package://marinero_simulations/robot_description/meshes/Wheel.stl" scale="1.0 1.0 1.0" />
             </geometry>
             <material name="black"/>
@@ -224,5 +224,5 @@
             <origin xyz="0 0 0.1466" rpy="0 0 ${pi/2}"/>
             <geometry>
-                <mesh filename="file:///home/albert/marinero_ws/src/marinero_simulations/robot_description/meshes/Wheel_Assembly.stl"  scale="1.0 1.0 1.0" />
+                <mesh filename="package://marinero_simulations/robot_description/meshes/Wheel_Assembly.stl"  scale="1.0 1.0 1.0" />
             </geometry>
             <material name="dark" />
@@ -266,5 +266,5 @@
             <origin xyz="0 0 0" rpy="0 0 0"/>
             <geometry>
-                <mesh filename="file:///home/albert/marinero_ws/src/marinero_simulations/robot_description/meshes/Wheel.stl" scale="1.0 1.0 1.0" />
+                <mesh filename="package://marinero_simulations/robot_description/meshes/Wheel.stl" scale="1.0 1.0 1.0" />
             </geometry>
             <material name="black"/>
@@ -301,5 +301,5 @@
             <origin xyz="0 0 0.1466" rpy="0 0 ${pi/2}"/>
             <geometry>
-                <mesh filename="file:///home/albert/marinero_ws/src/marinero_simulations/robot_description/meshes/Wheel_Assembly.stl"  scale="1.0 1.0 1.0" />
+                <mesh filename="package://marinero_simulations/robot_description/meshes/Wheel_Assembly.stl"  scale="1.0 1.0 1.0" />
             </geometry>
             <material name="dark" />
@@ -343,5 +343,5 @@
             <origin xyz="0 0 0" rpy="0 0 0"/>
             <geometry>
-                <mesh filename="file:///home/albert/marinero_ws/src/marinero_simulations/robot_description/meshes/Wheel.stl" scale="1.0 1.0 1.0" />
+                <mesh filename="package://marinero_simulations/robot_description/meshes/Wheel.stl" scale="1.0 1.0 1.0" />
             </geometry>
             <material name="black"/>

File: robot_description/ros2_control.xacro (robot description, xacro)
@@ -129,5 +129,5 @@
     <gazebo>
         <plugin name="gazebo_ros2_control" filename="libgazebo_ros2_control.so">
-            <parameters>/home/albert/marinero_ws/install/marinero_simulations/share/marinero_simulations/config/controllers.yaml</parameters>
+            <parameters>$(find marinero_simulations)/config/controllers.yaml</parameters>
         </plugin>
     </gazebo>
@@ -137,5 +137,5 @@
                 <remapping>~/out:=/joint_states</remapping>
             </ros>
-            <update_rate>500.0</update_rate>
+            <update_rate>200</update_rate>
             <joint_name>fl_rotation_joint</joint_name>
             <joint_name>fr_rotation_joint</joint_name>
@@ -159,5 +159,5 @@
             <frame_name>map</frame_name>
             <body_name>base_link</body_name>
-            <update_rate>150</update_rate>
+            <update_rate>100</update_rate>
             <gaussian_noise>0.01</gaussian_noise>
         </plugin>
