Commit message: Update to ros_jazzy on VB

File: robot_description/gazebo_control.xacro (robot description, xacro)
@@ -11,5 +11,4 @@
         <kd>10.0</kd>
         <fdir1>0 0 1</fdir1>
-        <material>Gazebo/Black</material>
     </gazebo>
     <gazebo reference="fr_wheel">
@@ -19,5 +18,4 @@
         <kd>10.0</kd>
         <fdir1>0 0 1</fdir1>
-        <material>Gazebo/Black</material>
     </gazebo>
     <gazebo reference="rl_wheel">
@@ -27,5 +25,4 @@
         <kd>10.0</kd>
         <fdir1>0 0 1</fdir1>
-        <material>Gazebo/Black</material>
     </gazebo>
     <gazebo reference="rr_wheel">
@@ -35,5 +32,4 @@
         <kd>10.0</kd>
         <fdir1>0 0 1</fdir1>
-        <material>Gazebo/Black</material>
     </gazebo>
     <gazebo reference="fl_axle_link">
@@ -42,5 +38,4 @@
         <kp>1e10</kp>
         <kd>10.0</kd>
-        <material>Gazebo/DarkGrey</material>
     </gazebo>
     <gazebo reference="fr_axle_link">
@@ -49,5 +44,4 @@
         <kp>1e10</kp>
         <kd>10.0</kd>
-        <material>Gazebo/DarkGrey</material>
     </gazebo>
     <gazebo reference="rl_axle_link">
@@ -56,5 +50,4 @@
         <kp>1e10</kp>
         <kd>10.0</kd>
-        <material>Gazebo/DarkGrey</material>
     </gazebo>
     <gazebo reference="rr_axle_link">
@@ -63,5 +56,4 @@
         <kp>1e10</kp>
         <kd>10.0</kd>
-        <material>Gazebo/DarkGrey</material>
     </gazebo>
     <gazebo reference="camera_base">
@@ -70,19 +62,10 @@
         <kp>5e10</kp>
         <kd>10.0</kd>
-        <material>Gazebo/DarkGrey</material>
     </gazebo>
-    <gazebo reference="left_camera_link">
-        <material>Gazebo/Grey</material>
-    </gazebo>
-    <gazebo reference="right_camera_link">
-        <material>Gazebo/Grey</material>
-    </gazebo>
-    <gazebo reference="lidar_link">
-        <material>Gazebo/Grey</material>
-    </gazebo>
+    <gazebo reference="left_camera_link"></gazebo>
+    <gazebo reference="right_camera_link"></gazebo>
+    <gazebo reference="lidar_link"></gazebo>
     <gazebo>
-        <plugin name="skid_steer_drive" filename="libgazebo_ros_diff_drive.so">
-            <!-- Update rate -->
-            <update_rate>100</update_rate>
+        <plugin filename="gz-sim-diff-drive-system" name="gz::sim::systems::DiffDrive">
             <!-- Number of wheel pairs -->
             <num_wheel_pairs>2</num_wheel_pairs>
@@ -95,27 +78,26 @@
             <wheel_separation>0.425</wheel_separation>
             <wheel_separation>0.425</wheel_separation>
-            <wheel_diameter>0.2032</wheel_diameter>
-            <wheel_diameter>0.2032</wheel_diameter>
+            <wheel_radius>0.1016</wheel_radius>
+            <wheel_radius>0.1016</wheel_radius>
             <!-- limits -->
-            <max_wheel_torque>100.0</max_wheel_torque>
-            <max_wheel_acceleration>7.0</max_wheel_acceleration>
+            <max_wheel_torque>20.0</max_wheel_torque>
+            <max_wheel_acceleration>10.0</max_wheel_acceleration>
+            <max_linear_acceleration>1.0</max_linear_acceleration>
             <!-- output -->
-            <publish_odom>true</publish_odom>
-            <publish_odom_tf>true</publish_odom_tf>
-            <publish_wheel_tf>true</publish_wheel_tf>
-            <odometry_frame>odom</odometry_frame>
-            <robot_base_frame>base_link</robot_base_frame>
-            <ros>
-                <remapping>/odom:=/marinero/odom</remapping>
-            </ros>
-            <covariance_x>0.001</covariance_x>
-            <covariance_y>0.001</covariance_y>
-            <covariance_yaw>0.01</covariance_yaw>
+            <topic>/cmd_vel</topic>
+            <odom_topic>/marinero/odom</odom_topic>
+            <frame_id>odom</frame_id>
+            <child_frame_id>base_link</child_frame_id>
+            <odom_publisher_frequency>50</odom_publisher_frequency>
+            <tf_topic>/tf</tf_topic>
         </plugin>
     </gazebo>
     <gazebo>
-        <plugin name="gazebo_ros_joint_state_publisher"
-            filename="libgazebo_ros_joint_state_publisher.so">
-            <update_rate>100</update_rate>
+        <plugin filename="gz-sim-joint-state-publisher-system" name="gz::sim::systems::JointStatePublisher">
+            <topic>/joint_states</topic>
+            <joint_name>fl_wheel_joint</joint_name>
+            <joint_name>fr_wheel_joint</joint_name>
+            <joint_name>rl_wheel_joint</joint_name>
+            <joint_name>rr_wheel_joint</joint_name>
             <joint_name>camera_base_joint</joint_name>
             <joint_name>left_camera_joint</joint_name>
@@ -123,9 +105,9 @@
         </plugin>
     </gazebo>
-    <gazebo>
+    <!-- <gazebo>
         <plugin name="gazebo_ros_joint_pose_trajectory"
             filename="libgazebo_ros_joint_pose_trajectory.so">
             <update_rate>100</update_rate>
         </plugin>
-    </gazebo>
+    </gazebo> -->
 </robot>

File: robot_description/imu.xacro (robot description, xacro)
@@ -20,26 +20,54 @@
             </geometry>
         </collision>
-    </link>
-    <gazebo reference="imu_link">
-        <gravity>true</gravity>
         <sensor name="imu_sensor" type="imu">
             <always_on>true</always_on>
             <update_rate>100</update_rate>
             <visualize>true</visualize>
-            <plugin filename="libgazebo_ros_imu_sensor.so" name="imu_plugin">
-                <ros>
-                    <remapping>~/out:=/marinero/imu_sensor</remapping>
-                </ros>
-                <body_name>imu_link</body_name>
-                <update_rate_hz>10.0</update_rate_hz>
-                <gaussian_noise>0.0</gaussian_noise>
-                <xyz_offset>0 0 0</xyz_offset>
-                <rpy_offset>0 0 0</rpy_offset>
-                <frame_name>imu_link</frame_name>
-                <initial_orientation_as_reference>false</initial_orientation_as_reference>
-            </plugin>
-            <pose>0 0 0 0 0 0</pose>
+            <topic>marinero/imu_sensor</topic>
+            <gz_frame_id>imu_link</gz_frame_id>
+            <imu>
+                <angular_velocity>
+                    <x>
+                        <noise type="gaussian">
+                            <mean>0.0</mean>
+                            <stddev>2e-4</stddev>
+                        </noise>
+                    </x>
+                    <y>
+                        <noise type="gaussian">
+                            <mean>0.0</mean>
+                            <stddev>2e-4</stddev>
+                        </noise>
+                    </y>
+                    <z>
+                        <noise type="gaussian">
+                            <mean>0.0</mean>
+                            <stddev>2e-4</stddev>
+                        </noise>
+                    </z>
+                </angular_velocity>
+                <linear_acceleration>
+                    <x>
+                        <noise type="gaussian">
+                            <mean>0.0</mean>
+                            <stddev>1.7e-2</stddev>
+                        </noise>
+                    </x>
+                    <y>
+                        <noise type="gaussian">
+                            <mean>0.0</mean>
+                            <stddev>1.7e-2</stddev>
+                        </noise>
+                    </y>
+                    <z>
+                        <noise type="gaussian">
+                            <mean>0.0</mean>
+                            <stddev>1.7e-2</stddev>
+                        </noise>
+                    </z>
+                </linear_acceleration>
+            </imu>
         </sensor>
-    </gazebo>
+    </link>
     <joint name="gps_joint" type="fixed">
         <parent link="base_link"/>
@@ -61,15 +89,12 @@
             </geometry>
         </collision>
-    </link>
-    <gazebo reference="gps_link">
         <sensor name="gps_sensor" type="gps">
             <always_on>true</always_on>
             <update_rate>10</update_rate>
-            <plugin name="my_gps_plugin" filename="libgazebo_ros_gps_sensor.so">
-                <ros>
-                    <remapping>~/out:=/marinero/gps_sensor</remapping>
-                </ros>
-            </plugin>
+            <topic>marinero/gps_sensor</topic>
+            <gz_frame_id>gps_link</gz_frame_id>
         </sensor>
-    </gazebo>
+    </link>
+    <gazebo reference="imu_link"></gazebo>
+    <gazebo reference="gps_link"></gazebo>
 </robot>

File: robot_description/lidar.xacro (robot description, xacro)
@@ -41,5 +41,28 @@
         <child link="lidar_2D_link"/>
     </joint>
-    <link name="lidar_2D_link"></link>
+    <link name="lidar_2D_link">
+        <sensor name="2D_lidar" type="gpu_lidar">
+            <pose>0 0 0 0 0 0</pose>
+            <update_rate>10</update_rate>
+            <visualize>false</visualize>
+            <topic>scan</topic>
+            <gz_frame_id>lidar_2D_link</gz_frame_id>
+            <lidar>
+                <scan>
+                    <horizontal>
+                        <samples>720</samples>
+                        <resolution>1</resolution>
+                        <min_angle>-3.14</min_angle>
+                        <max_angle>3.14</max_angle>
+                    </horizontal>
+                </scan>
+                <range>
+                    <min>0.75</min>
+                    <max>15</max>
+                    <resolution>0.01</resolution>
+                </range>
+            </lidar>
+        </sensor>
+    </link>
     <joint name="lidar_3D_joint" type="fixed">
         <origin xyz="0.0 0.0 0.0" rpy="0.0 0.0 0.0"/>
@@ -47,12 +70,12 @@
         <child link="lidar_3D_link"/>
     </joint>
-    <link name="lidar_3D_link"></link>
-    <!-- 3D LIDAR -->
-    <gazebo reference="lidar_3D_link">
-        <sensor name="3D_lidar" type="gpu_ray">
+    <link name="lidar_3D_link">
+        <sensor name="3D_lidar" type="gpu_lidar">
             <pose>0 0 0 0 0 0</pose>
-            <update_rate>15.0</update_rate>
+            <update_rate>10</update_rate>
             <visualize>false</visualize>
-            <ray>
+            <topic>lidar_3D/scan</topic>
+            <gz_frame_id>lidar_3D_link</gz_frame_id>
+            <lidar>
                 <scan>
                     <horizontal>
@@ -74,45 +97,8 @@
                     <resolution>0.001</resolution>
                 </range>
-            </ray>
-            <plugin name="laser_3D_plugin" filename="libgazebo_ros_ray_sensor.so">
-                <ros>
-                    <remapping>~/out:=/lidar_3D/scan</remapping>
-                </ros>
-                <update_rate>15.0</update_rate>
-                <output_type>sensor_msgs/PointCloud2</output_type>
-                <frame_name>lidar_3D_link</frame_name>
-            </plugin>
+            </lidar>
         </sensor>
-    </gazebo>
-    <!-- 2D LIDAR -->
-    <gazebo reference="lidar_2D_link">
-        <sensor name="2D_lidar" type="gpu_ray">
-            <pose> 0 0 0 0 0 0 </pose>
-            <update_rate>15.0</update_rate>
-            <visualize>false</visualize>
-            <ray>
-                <scan>
-                    <horizontal>
-                        <samples>720</samples>
-                        <resolution>1</resolution>
-                        <min_angle>-3.14</min_angle>
-                        <max_angle>3.14</max_angle>
-                    </horizontal>
-                </scan>
-                <range>
-                    <min>0.75</min>
-                    <max>15</max>
-                    <resolution>0.01</resolution>
-                </range>
-            </ray>
-            <plugin name="laser_2D_plugin" filename="libgazebo_ros_ray_sensor.so">
-                <ros>
-                    <remapping>~/out:=/scan</remapping>
-                </ros>
-                <update_rate>15.0</update_rate>
-                <output_type>sensor_msgs/LaserScan</output_type>
-                <frame_name>lidar_2D_link</frame_name>
-            </plugin>
-        </sensor>
-    </gazebo>
+    </link>
+    <gazebo reference="lidar_2D_link"></gazebo>
+    <gazebo reference="lidar_3D_link"></gazebo>
 </robot>

File: robot_description/marinero_camera.xacro (robot description, xacro)
@@ -82,5 +82,26 @@
         <child link="right_camera_depth_frame"/>
     </joint>
-    <link name="right_camera_depth_frame"></link>
+    <link name="right_camera_depth_frame">
+        <sensor name="right_depth_camera" type="depth">
+            <always_on>true</always_on>
+            <visualize>true</visualize>
+            <update_rate>50</update_rate>
+            <topic>right_depth_camera/image_raw</topic>
+            <gz_frame_id>right_camera_depth_frame</gz_frame_id>
+            <camera name="right_dep_cam">
+                <camera_info_topic>right_depth_camera/camera_info</camera_info_topic>
+                <horizontal_fov>1.3962634</horizontal_fov>
+                <image>
+                    <width>640</width>
+                    <height>480</height>
+                    <format>B8G8R8</format>
+                </image>
+                <clip>
+                    <near>0.025</near>
+                    <far>20</far>
+                </clip>
+            </camera>
+        </sensor>
+    </link>
     <!-- LEFT CAMERA -->
     <joint name="left_camera_joint" type="revolute">
@@ -129,11 +150,13 @@
         <child link="left_camera_depth_frame"/>
     </joint>
-    <link name="left_camera_depth_frame"></link>
-    <!-- GAZEBO PLUGINS -->
-    <gazebo reference="right_camera_center_link">
-        <sensor name="right_depth_camera" type="depth">
-            <update_rate>50.0</update_rate>
-            <visualize>false</visualize>
+    <link name="left_camera_depth_frame">
+        <!-- <sensor name="left_depth_camera" type="depth">
+            <always_on>true</always_on>
+            <visualize>true</visualize>
+            <update_rate>50</update_rate>
+            <topic>left_depth_camera/image_raw</topic>
+            <gz_frame_id>left_camera_depth_frame</gz_frame_id>
             <camera name="right_dep_cam">
+                <camera_info_topic>left_depth_camera/camera_info</camera_info_topic>
                 <horizontal_fov>1.3962634</horizontal_fov>
                 <image>
@@ -147,36 +170,7 @@
                 </clip>
             </camera>
-            <plugin name="right_camera_controller" filename="libgazebo_ros_camera.so">
-                <frame_name>right_camera_depth_frame</frame_name>
-                <update_rate>50.0</update_rate>
-                <min_depth>0.025</min_depth>
-                <max_depth>20</max_depth>
-            </plugin>
-        </sensor>
-    </gazebo>
-    <!-- <gazebo reference="left_camera_center_link">
-        <sensor name="left_depth_camera" type="depth">
-            <update_rate>20</update_rate>
-            <visualize>false</visualize>
-            <camera name="left_dep_cam">
-                <horizontal_fov>1.3962634</horizontal_fov>
-                <image>
-                    <width>640</width>
-                    <height>480</height>
-                    <format>B8G8R8</format>
-                </image>
-                <clip>
-                    <near>0.1</near>
-                    <far>25</far>
-                </clip>
-            </camera>
-            <plugin name="left_camera_controller" filename="libgazebo_ros_camera.so">
-                <frame_name>left_camera_depth_frame</frame_name>
-                <imageTopicName>camera/image_left</imageTopicName>
-                <depthImageTopicName>camera/depth_image_left</depthImageTopicName>
-                <min_depth>0.1</min_depth>
-                <max_depth>25</max_depth>
-            </plugin>
-        </sensor>
-    </gazebo> -->
+        </sensor> -->
+    </link>
+    <gazebo reference="right_camera_center_link"></gazebo>
+    <gazebo reference="left_camera_center_link"></gazebo>
 </robot>

File: robot_description/ros2_control.xacro (robot description, xacro)
@@ -3,5 +3,5 @@
     <ros2_control name="GazeboSystem" type="system">
         <hardware>
-            <plugin>gazebo_ros2_control/GazeboSystem</plugin>
+            <plugin>gazebo_ros2_control/GazeboSimSystem</plugin>
         </hardware>
         <!-- ROTATION JOINTS -->
@@ -133,9 +133,7 @@
     </gazebo>
     <!-- <gazebo>
-        <plugin name="marinero_robot_joint_state" filename="libgazebo_ros_joint_state_publisher.so">
-            <ros>
-                <remapping>~/out:=/joint_states</remapping>
-            </ros>
-            <update_rate>200</update_rate>
+        <plugin filename="gz-sim-joint-state-publisher-system" name="gz::sim::systems::JointStatePublisher">
+            <topic>/joint_states</topic>
+            <update_rate>100</update_rate>
             <joint_name>fl_rotation_joint</joint_name>
             <joint_name>fr_rotation_joint</joint_name>
@@ -151,16 +149,4 @@
         </plugin>
     </gazebo> -->
-    <gazebo>
-        <plugin name="libgazebo_ros_p3d" filename="libgazebo_ros_p3d.so">
-            <ros>
-                <namespace>/</namespace>
-                <remapping>odom:=/marinero/odom</remapping>
-            </ros>
-            <frame_name>map</frame_name>
-            <body_name>base_link</body_name>
-            <update_rate>100</update_rate>
-            <gaussian_noise>0.01</gaussian_noise>
-        </plugin>
-    </gazebo>
     <gazebo reference="chassis">
         <mu1>1.0</mu1>
@@ -170,58 +156,44 @@
         <mu1>2.0</mu1>
         <mu2>2.0</mu2>
-        <material>Gazebo/Black</material>
     </gazebo>
     <gazebo reference="fr_wheel">
         <mu1>2.0</mu1>
         <mu2>2.0</mu2>
-        <material>Gazebo/Black</material>
     </gazebo>
     <gazebo reference="rl_wheel">
         <mu1>2.0</mu1>
         <mu2>2.0</mu2>
-        <material>Gazebo/Black</material>
     </gazebo>
     <gazebo reference="rr_wheel">
         <mu1>2.0</mu1>
         <mu2>2.0</mu2>
-        <material>Gazebo/Black</material>
     </gazebo>
     <gazebo reference="fl_axle_link">
         <mu1>0.5</mu1>
         <mu2>0.5</mu2>
-        <material>Gazebo/DarkGrey</material>
     </gazebo>
     <gazebo reference="fr_axle_link">
         <mu1>0.5</mu1>
         <mu2>0.5</mu2>
-        <material>Gazebo/DarkGrey</material>
     </gazebo>
     <gazebo reference="rl_axle_link">
         <mu1>0.5</mu1>
         <mu2>0.5</mu2>
-        <material>Gazebo/DarkGrey</material>
     </gazebo>
     <gazebo reference="rr_axle_link">
         <mu1>0.5</mu1>
         <mu2>0.5</mu2>
-        <material>Gazebo/DarkGrey</material>
     </gazebo>
     <gazebo reference="camera_base">
         <mu1>5.0</mu1>
         <mu2>5.0</mu2>
-        <material>Gazebo/DarkGrey</material>
     </gazebo>
     <gazebo reference="left_camera_link">
         <mu1>5.0</mu1>
         <mu2>5.0</mu2>
-        <material>Gazebo/Grey</material>
     </gazebo>
     <gazebo reference="right_camera_link">
         <mu1>5.0</mu1>
         <mu2>5.0</mu2>
-        <material>Gazebo/Grey</material>
-    </gazebo>
-    <gazebo reference="lidar_link">
-        <material>Gazebo/Grey</material>
     </gazebo>
 </robot>
