Commit message: Update 06_03_1

File: robot_description/gazebo_control.xacro (robot description, xacro)
@@ -1,5 +1,5 @@
 <?xml version="1.0" ?>
 <robot xmlns:xacro="http://www.ros.org/wiki/xacro">
-    <gazebo reference="chassis">
+    <!-- <gazebo reference="chassis">
         <mu1>1.0</mu1>
         <mu2>1.0</mu2>
@@ -62,8 +62,5 @@
         <kp>5e10</kp>
         <kd>10.0</kd>
-    </gazebo>
-    <gazebo reference="left_camera_link"></gazebo>
-    <gazebo reference="right_camera_link"></gazebo>
-    <gazebo reference="lidar_link"></gazebo>
+    </gazebo> -->
     <gazebo>
         <plugin filename="gz-sim-diff-drive-system" name="gz::sim::systems::DiffDrive">
@@ -81,18 +78,70 @@
             <wheel_radius>0.1016</wheel_radius>
             <!-- limits -->
-            <max_wheel_torque>20.0</max_wheel_torque>
-            <max_wheel_acceleration>10.0</max_wheel_acceleration>
-            <max_linear_acceleration>1.0</max_linear_acceleration>
+            <max_wheel_torque>50.0</max_wheel_torque>
+            <max_wheel_acceleration>5.0</max_wheel_acceleration>
+            <max_linear_acceleration>5.0</max_linear_acceleration>
+            <!-- input -->
+            <topic>cmd_vel_stamped</topic>
             <!-- output -->
-            <topic>/cmd_vel</topic>
-            <odom_topic>/marinero/odom</odom_topic>
+            <odom_topic>marinero/odom</odom_topic>
             <frame_id>odom</frame_id>
             <child_frame_id>base_link</child_frame_id>
-            <odom_publisher_frequency>50</odom_publisher_frequency>
+            <odom_publisher_frequency>100</odom_publisher_frequency>
             <tf_topic>/tf</tf_topic>
         </plugin>
+        <plugin filename="gz_ros2_control-system" name="gz_ros2_control::GazeboSimROS2ControlPlugin" >
+            <parameters>$(find marinero_simulations)/config/camera_controller.yaml</parameters>
+        </plugin>
+        <plugin filename="gz-sim-joint-state-publisher-system" name="gz::sim::systems::JointStatePublisher">
+            <topic>joint_states</topic>
+            <joint_name>fl_wheel_joint</joint_name>
+            <joint_name>fr_wheel_joint</joint_name>
+            <joint_name>rl_wheel_joint</joint_name>
+            <joint_name>rr_wheel_joint</joint_name>
+            <joint_name>camera_base_joint</joint_name>
+            <joint_name>left_camera_joint</joint_name>
+            <joint_name>right_camera_joint</joint_name>
+        </plugin>
     </gazebo>
-    <gazebo>
-        <plugin filename="gz-sim-joint-state-publisher-system" name="gz::sim::systems::JointStatePublisher">
+    <ros2_control name="GazeboSimSystem" type="system">
+        <hardware>
+            <plugin>gz_ros2_control/GazeboSimSystem</plugin>
+        </hardware>
+        <joint name="camera_base_joint">
+            <command_interface name="position">
+                <param name="min">-1.57</param>
+                <param name="max">1.57</param>
+            </command_interface>
+            <state_interface name="position">
+                <param name="initial_value">0.0</param>
+            </state_interface>
+            <state_interface name="velocity" />
+            <state_interface name="effort" />
+        </joint>
+        <joint name="right_camera_joint">
+            <command_interface name="position">
+                <param name="min">-1.57</param>
+                <param name="max">1.57</param>
+            </command_interface>
+            <state_interface name="position">
+                <param name="initial_value">1.6</param>
+            </state_interface>
+            <state_interface name="velocity" />
+            <state_interface name="effort" />
+        </joint>
+        <joint name="left_camera_joint">
+            <command_interface name="position">
+                <param name="min">-1.57</param>
+                <param name="max">1.57</param>
+            </command_interface>
+            <state_interface name="position">
+                <param name="initial_value">1.5</param>
+            </state_interface>
+            <state_interface name="velocity" />
+            <state_interface name="effort" />
+        </joint>
+    </ros2_control>
+    <!-- <gazebo>
+        <plugin filename="gz-sim-joint-state-broadcaster-system" name="gz::sim::systems::JointStateBroadcaster">
             <topic>/joint_states</topic>
             <joint_name>fl_wheel_joint</joint_name>
@@ -104,10 +153,4 @@
             <joint_name>right_camera_joint</joint_name>
         </plugin>
-    </gazebo>
-    <!-- <gazebo>
-        <plugin name="gazebo_ros_joint_pose_trajectory"
-            filename="libgazebo_ros_joint_pose_trajectory.so">
-            <update_rate>100</update_rate>
-        </plugin>
     </gazebo> -->
 </robot>

File: robot_description/lidar.xacro (robot description, xacro)
@@ -46,6 +46,4 @@
             <update_rate>10</update_rate>
             <visualize>false</visualize>
-            <topic>scan</topic>
-            <gz_frame_id>lidar_2D_link</gz_frame_id>
             <lidar>
                 <scan>
@@ -63,4 +61,6 @@
                 </range>
             </lidar>
+            <topic>scan</topic>
+            <gz_frame_id>lidar_2D_link</gz_frame_id>
         </sensor>
     </link>
@@ -75,6 +75,4 @@
             <update_rate>10</update_rate>
             <visualize>false</visualize>
-            <topic>lidar_3D/scan</topic>
-            <gz_frame_id>lidar_3D_link</gz_frame_id>
             <lidar>
                 <scan>
@@ -98,4 +96,6 @@
                 </range>
             </lidar>
+            <topic>lidar_3D/scan</topic>
+            <gz_frame_id>lidar_3D_link</gz_frame_id>
         </sensor>
     </link>

File: robot_description/marinero_camera.xacro (robot description, xacro)
@@ -47,5 +47,5 @@
             effort="100"
             velocity="100" />
-        <dynamics damping="10.0" friction="10.0" />
+        <dynamics damping="10.0" friction="5.0" />
     </joint>
     <link name="right_camera_link">
@@ -83,10 +83,9 @@
     </joint>
     <link name="right_camera_depth_frame">
-        <sensor name="right_depth_camera" type="depth">
+        <pose>0 0 0 0 0 0</pose>
+        <sensor name="right_depth_camera" type="camera">
             <always_on>true</always_on>
             <visualize>true</visualize>
             <update_rate>50</update_rate>
-            <topic>right_depth_camera/image_raw</topic>
-            <gz_frame_id>right_camera_depth_frame</gz_frame_id>
             <camera name="right_dep_cam">
                 <camera_info_topic>right_depth_camera/camera_info</camera_info_topic>
@@ -102,4 +101,6 @@
                 </clip>
             </camera>
+            <topic>right_depth_camera/image_raw</topic>
+            <gz_frame_id>right_camera_depth_frame</gz_frame_id>
         </sensor>
     </link>
@@ -151,10 +152,9 @@
     </joint>
     <link name="left_camera_depth_frame">
-        <!-- <sensor name="left_depth_camera" type="depth">
+        <!-- <pose>0 0 0 0 0 0</pose>
+        <sensor name="left_depth_camera" type="depth">
             <always_on>true</always_on>
             <visualize>true</visualize>
             <update_rate>50</update_rate>
-            <topic>left_depth_camera/image_raw</topic>
-            <gz_frame_id>left_camera_depth_frame</gz_frame_id>
             <camera name="right_dep_cam">
                 <camera_info_topic>left_depth_camera/camera_info</camera_info_topic>
@@ -170,7 +170,9 @@
                 </clip>
             </camera>
+            <topic>left_depth_camera/image_raw</topic>
+            <gz_frame_id>left_camera_depth_frame</gz_frame_id>
         </sensor> -->
     </link>
-    <gazebo reference="right_camera_center_link"></gazebo>
-    <gazebo reference="left_camera_center_link"></gazebo>
+    <gazebo reference="right_camera_depth_frame"></gazebo>
+    <gazebo reference="left_camera_depth_frame"></gazebo>
 </robot>

File: robot_description/robot_core.xacro (robot description, xacro)
@@ -95,6 +95,5 @@
         <child link="fl_wheel" />
         <axis xyz="0 0 1" />
-        <dynamics damping="0.1"/>
-        <limit effort="50" velocity="20"/>
+        <limit effort="100" velocity="20"/>
     </joint>
     <link name="fl_wheel">
@@ -164,6 +163,5 @@
         <child link="fr_wheel" />
         <axis xyz="0 0 -1" />
-        <dynamics damping="0.1"/>
-        <limit effort="50" velocity="20"/>
+        <limit effort="100" velocity="20"/>
     </joint>
     <link name="fr_wheel">
@@ -232,6 +230,5 @@
         <child link="rl_wheel" />
         <axis xyz="0 0 1" />
-        <dynamics damping="0.1"/>
-        <limit effort="50" velocity="20"/>
+        <limit effort="100" velocity="20"/>
     </joint>
     <link name="rl_wheel">
@@ -300,6 +297,5 @@
         <child link="rr_wheel" />
         <axis xyz="0 0 -1" />
-        <dynamics damping="0.1"/>
-        <limit effort="50" velocity="20"/>
+        <limit effort="100" velocity="20"/>
     </joint>
     <link name="rr_wheel">
