Commit message: Update 26_06

File: robot_description/SUNELL_camera.xacro (robot description, xacro)
@@ -5,5 +5,5 @@
         <parent link="chassis" />
         <child link="camera_base" />
-        <axis xyz="0 0 -1" />
+        <axis xyz="0 0 1" />
         <limit
             upper="${pi}"
@@ -140,5 +140,5 @@
                 <clip>
                     <near>0.05</near>
-                    <far>10</far>
+                    <far>20</far>
                 </clip>
             </camera>
@@ -147,5 +147,5 @@
                 <update_rate>20</update_rate>
                 <min_depth>0.05</min_depth>
-                <max_depth>10</max_depth>
+                <max_depth>20</max_depth>
             </plugin>
         </sensor>

File: robot_description/lidar.xacro (robot description, xacro)
@@ -64,5 +64,5 @@
                 <range>
                     <min>0.25</min>
-                    <max>5.0</max>
+                    <max>10.0</max>
                     <resolution>0.001</resolution>
                 </range>

File: robot_description/robot_core_4WIS4WID.xacro (robot description, xacro)
@@ -54,5 +54,5 @@
         <parent link="base_link" />
         <child link="fl_axle_link" />
-        <axis xyz="0 0 -1" />
+        <axis xyz="0 0 1" />
         <limit
             upper="${pi/2}"
@@ -130,5 +130,5 @@
         <parent link="base_link" />
         <child link="fr_axle_link" />
-        <axis xyz="0 0 -1" />
+        <axis xyz="0 0 1" />
         <limit
             upper="${pi/2}"
@@ -206,5 +206,5 @@
         <parent link="base_link" />
         <child link="rl_axle_link" />
-        <axis xyz="0 0 -1" />
+        <axis xyz="0 0 1" />
         <limit
             upper="${pi/2}"
@@ -282,5 +282,5 @@
         <parent link="base_link" />
         <child link="rr_axle_link" />
-        <axis xyz="0 0 -1" />
+        <axis xyz="0 0 1" />
         <limit
             upper="${pi/2}"

File: robot_description/robot_core_SKID_STEER.xacro (robot description, xacro)
@@ -54,5 +54,4 @@
         <parent link="base_link" />
         <child link="fl_axle_link" />
-        <axis xyz="0 0 -1" />
     </joint>
     <link name="fl_axle_link">

File: robot_description/rsp_marinero_robot.urdf.xacro (robot description, xacro)
@@ -5,4 +5,5 @@
   <xacro:include filename="lidar.xacro" />
   <xacro:include filename="marinero_camera.xacro" />
+  <xacro:include filename="SUNELL_camera.xacro" />
   <xacro:include filename="robot_core_4WIS4WID.xacro" />
 </robot>
